File: y_arena_valve_controller.kicad_pcb (KiCad board)
At the start: 2 copper layers, 74.9 x 80.6 mm, 105 parts, among them P1 PWR_JACK_2.1x5.5_SMD_RA, SW1 SPDT_SLIDE_500A_SM, U1 DRV103, U2 DRV103, U3 DRV103, U4 DRV103, U5 DRV103, U6 DRV103, U7 DRV103, U8 DRV103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

Commit message: Rename VALVE lines from VALVE_0 -> ARM_0_VALVE_0
Connections:
- net /VALVE_0 renamed /ARM_0_VALVE_0
- net /VALVE_1 renamed /ARM_0_VALVE_1
- net /VALVE_2 renamed /ARM_0_VALVE_2
- net /VALVE_3 renamed /ARM_1_VALVE_0
- net /VALVE_4 renamed /ARM_1_VALVE_1
- net /VALVE_5 renamed /ARM_1_VALVE_2
- net /VALVE_6 renamed /ARM_2_VALVE_0
- net /VALVE_7 renamed /ARM_2_VALVE_1
- net /VALVE_8 renamed /ARM_2_VALVE_2
Changed lines of the file:
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@@
   )
   (net 0 "")
-  (net 1 /VALVE_0)
-  (net 2 /VALVE_1)
-  (net 3 /VALVE_2)
-  (net 4 /VALVE_3)
-  (net 5 /VALVE_4)
-  (net 6 /VALVE_5)
-  (net 7 /VALVE_6)
-  (net 8 /VALVE_7)
-  (net 9 /VALVE_8)
+  (net 1 /ARM_0_VALVE_0)
+  (net 2 /ARM_0_VALVE_1)
+  (net 3 /ARM_0_VALVE_2)
+  (net 4 /ARM_1_VALVE_0)
+  (net 5 /ARM_1_VALVE_1)
+  (net 6 /ARM_1_VALVE_2)
+  (net 7 /ARM_2_VALVE_0)
+  (net 8 /ARM_2_VALVE_1)
+  (net 9 /ARM_2_VALVE_2)
   (net 10 VAA)
   (net 11 GND)
@@
     (diff_pair_width 0.254)
     (diff_pair_gap 0.254)
-    (add_net /VALVE_0)
-    (add_net /VALVE_1)
-    (add_net /VALVE_2)
-    (add_net /VALVE_3)
-    (add_net /VALVE_4)
-    (add_net /VALVE_5)
-    (add_net /VALVE_6)
-    (add_net /VALVE_7)
-    (add_net /VALVE_8)
+    (add_net /ARM_0_VALVE_0)
+    (add_net /ARM_0_VALVE_1)
+    (add_net /ARM_0_VALVE_2)
+    (add_net /ARM_1_VALVE_0)
+    (add_net /ARM_1_VALVE_1)
+    (add_net /ARM_1_VALVE_2)
+    (add_net /ARM_2_VALVE_0)
+    (add_net /ARM_2_VALVE_1)
+    (add_net /ARM_2_VALVE_2)
     (add_net /Vled)
     (add_net /valve_0/SH)
@@
     (pad 23 thru_hole oval (at 7.62 -8.89 180) (size 2.54 2.1844) (drill 1.5494) (layers *.Cu *.Mask))
     (pad 22 thru_hole oval (at 7.62 -6.35 180) (size 2.54 2.1844) (drill 1.5494) (layers *.Cu *.Mask)
-      (net 1 /VALVE_0))
+      (net 1 /ARM_0_VALVE_0))
     (pad 21 thru_hole oval (at 7.62 -3.81 180) (size 2.54 2.1844) (drill 1.5494) (layers *.Cu *.Mask)
-      (net 2 /VALVE_1))
+      (net 2 /ARM_0_VALVE_1))
     (pad 20 thru_hole oval (at 7.62 -1.27 180) (size 2.54 2.1844) (drill 1.5494) (layers *.Cu *.Mask)
-      (net 3 /VALVE_2))
+      (net 3 /ARM_0_VALVE_2))
     (pad 19 thru_hole oval (at 7.62 1.27 180) (size 2.54 2.1844) (drill 1.5494) (layers *.Cu *.Mask)
-      (net 4 /VALVE_3))
+      (net 4 /ARM_1_VALVE_0))
     (pad 18 thru_hole oval (at 7.62 3.81 180) (size 2.54 2.1844) (drill 1.5494) (layers *.Cu *.Mask)
-      (net 5 /VALVE_4))
+      (net 5 /ARM_1_VALVE_1))
     (pad 17 thru_hole oval (at 7.62 6.35 180) (size 2.54 2.1844) (drill 1.5494) (layers *.Cu *.Mask)
-      (net 6 /VALVE_5))
+      (net 6 /ARM_1_VALVE_2))
     (pad 16 thru_hole oval (at 7.62 8.89 180) (size 2.54 2.1844) (drill 1.5494) (layers *.Cu *.Mask)
-      (net 7 /VALVE_6))
+      (net 7 /ARM_2_VALVE_0))
     (pad 15 thru_hole oval (at 7.62 11.43 180) (size 2.54 2.1844) (drill 1.5494) (layers *.Cu *.Mask)
-      (net 8 /VALVE_7))
+      (net 8 /ARM_2_VALVE_1))
     (pad 14 thru_hole oval (at 7.62 13.97 180) (size 2.54 2.1844) (drill 1.5494) (layers *.Cu *.Mask)
-      (net 9 /VALVE_8))
+      (net 9 /ARM_2_VALVE_2))
     (pad 13 thru_hole oval (at 7.62 16.51 180) (size 2.54 2.1844) (drill 1.5494) (layers *.Cu *.Mask))
     (pad 12 thru_hole oval (at -7.62 16.51 180) (size 2.54 2.1844) (drill 1.5494) (layers *.Cu *.Mask))
@@
     (fp_circle (center -0.889 1.651) (end -0.508 1.651) (layer B.SilkS) (width 0.381))
     (pad 8 smd rect (at 2.6924 1.905 270) (size 0.59944 1.5494) (layers B.Cu B.Paste B.Mask)
-      (net 1 /VALVE_0))
+      (net 1 /ARM_0_VALVE_0))
     (pad 7 smd rect (at 2.6924 0.635 270) (size 0.59944 1.5494) (layers B.Cu B.Paste B.Mask))
     (pad 6 smd rect (at 2.6924 -0.635 270) (size 0.59944 1.5494) (layers B.Cu B.Paste B.Mask)
@@
     (fp_circle (center -0.889 1.651) (end -0.508 1.651) (layer B.SilkS) (width 0.381))
     (pad 8 smd rect (at 2.6924 1.905 270) (size 0.59944 1.5494) (layers B.Cu B.Paste B.Mask)
-      (net 2 /VALVE_1))
+      (net 2 /ARM_0_VALVE_1))
     (pad 7 smd rect (at 2.6924 0.635 270) (size 0.59944 1.5494) (layers B.Cu B.Paste B.Mask))
     (pad 6 smd rect (at 2.6924 -0.635 270) (size 0.59944 1.5494) (layers B.Cu B.Paste B.Mask)
@@
     (fp_circle (center -0.889 1.651) (end -0.508 1.651) (layer B.SilkS) (width 0.381))
     (pad 8 smd rect (at 2.6924 1.905 270) (size 0.59944 1.5494) (layers B.Cu B.Paste B.Mask)
-      (net 3 /VALVE_2))
+      (net 3 /ARM_0_VALVE_2))
     (pad 7 smd rect (at 2.6924 0.635 270) (size 0.59944 1.5494) (layers B.Cu B.Paste B.Mask))
     (pad 6 smd rect (at 2.6924 -0.635 270) (size 0.59944 1.5494) (layers B.Cu B.Paste B.Mask)
@@
     (fp_circle (center -0.889 1.651) (end -0.508 1.651) (layer B.SilkS) (width 0.381))
     (pad 8 smd rect (at 2.6924 1.905 270) (size 0.59944 1.5494) (layers B.Cu B.Paste B.Mask)
-      (net 4 /VALVE_3))
+      (net 4 /ARM_1_VALVE_0))
     (pad 7 smd rect (at 2.6924 0.635 270) (size 0.59944 1.5494) (layers B.Cu B.Paste B.Mask))
     (pad 6 smd rect (at 2.6924 -0.635 270) (size 0.59944 1.5494) (layers B.Cu B.Paste B.Mask)
@@
     (fp_circle (center -0.889 1.651) (end -0.508 1.651) (layer B.SilkS) (width 0.381))
     (pad 8 smd rect (at 2.6924 1.905 270) (size 0.59944 1.5494) (layers B.Cu B.Paste B.Mask)
-      (net 5 /VALVE_4))
+      (net 5 /ARM_1_VALVE_1))
     (pad 7 smd rect (at 2.6924 0.635 270) (size 0.59944 1.5494) (layers B.Cu B.Paste B.Mask))
     (pad 6 smd rect (at 2.6924 -0.635 270) (size 0.59944 1.5494) (layers B.Cu B.Paste B.Mask)
@@
     (fp_circle (center -0.889 1.651) (end -0.508 1.651) (layer B.SilkS) (width 0.381))
     (pad 8 smd rect (at 2.6924 1.905 270) (size 0.59944 1.5494) (layers B.Cu B.Paste B.Mask)
-      (net 6 /VALVE_5))
+      (net 6 /ARM_1_VALVE_2))
     (pad 7 smd rect (at 2.6924 0.635 270) (size 0.59944 1.5494) (layers B.Cu B.Paste B.Mask))
     (pad 6 smd rect (at 2.6924 -0.635 270) (size 0.59944 1.5494) (layers B.Cu B.Paste B.Mask)
@@
     (fp_circle (center -0.889 1.651) (end -0.508 1.651) (layer B.SilkS) (width 0.381))
     (pad 8 smd rect (at 2.6924 1.905 270) (size 0.59944 1.5494) (layers B.Cu B.Paste B.Mask)
-      (net 7 /VALVE_6))
+      (net 7 /ARM_2_VALVE_0))
     (pad 7 smd rect (at 2.6924 0.635 270) (size 0.59944 1.5494) (layers B.Cu B.Paste B.Mask))
     (pad 6 smd rect (at 2.6924 -0.635 270) (size 0.59944 1.5494) (layers B.Cu B.Paste B.Mask)
@@
     (fp_circle (center -0.889 1.651) (end -0.508 1.651) (layer B.SilkS) (width 0.381))
     (pad 8 smd rect (at 2.6924 1.905 270) (size 0.59944 1.5494) (layers B.Cu B.Paste B.Mask)
-      (net 8 /VALVE_7))
+      (net 8 /ARM_2_VALVE_1))
     (pad 7 smd rect (at 2.6924 0.635 270) (size 0.59944 1.5494) (layers B.Cu B.Paste B.Mask))
     (pad 6 smd rect (at 2.6924 -0.635 270) (size 0.59944 1.5494) (layers B.Cu B.Paste B.Mask)
@@
     (fp_circle (center -0.889 1.651) (end -0.508 1.651) (layer B.SilkS) (width 0.381))
     (pad 8 smd rect (at 2.6924 1.905 270) (size 0.59944 1.5494) (layers B.Cu B.Paste B.Mask)
-      (net 9 /VALVE_8))
+      (net 9 /ARM_2_VALVE_2))
     (pad 7 smd rect (at 2.6924 0.635 270) (size 0.59944 1.5494) (layers B.Cu B.Paste B.Mask))
     (pad 6 smd rect (at 2.6924 -0.635 270) (size 0.59944 1.5494) (layers B.Cu B.Paste B.Mask)
