File: y_arena_odor_controller.kicad_pcb (KiCad board)
At the start: 2 copper layers, 74.9 x 80.6 mm, 105 parts, among them P1 PWR_JACK_2.1x5.5_SMD_RA, SW1 SPDT_SLIDE_500A_SM, U1 DRV103, U2 DRV103, U3 DRV103, U4 DRV103, U5 DRV103, U6 DRV103, U7 DRV103, U8 DRV103, U9 DRV103

Commit message: Complete v1.3
Parts:
- C1: footprint y_arena_valve_controller:SM0805 -> y_arena_odor_controller:SM0805
- C10, C12, C14, C16, C18, C2, C4, C6, C8, D10, D11, D12, D13, D14, D15, D16, D17, D18, D19, D20, D3, D4, D5, D6, D7, D8, D9: footprint valve_spike_hold:SM0402_POL -> odor_spike_hold:SM0402_POL
- C11, C13, C15, C17, C19, C3, C5, C7, C9, R10, R11, R12, R13, R14, R15, R16, R17, R18, R19, R2, R20, R21, R22, R23, R24, R25, R26, R27, R28, R3, R4, R5, R6, R7, R8, R9: footprint valve_spike_hold:SM0402 -> odor_spike_hold:SM0402
- D1: footprint y_arena_valve_controller:CFP15 -> y_arena_odor_controller:CFP15
- D2: footprint y_arena_valve_controller:SM0402_POL -> y_arena_odor_controller:SM0402_POL
- FID1, FID2, FID3, FID4: footprint y_arena_valve_controller:FIDUCIAL -> y_arena_odor_controller:FIDUCIAL
- L1: footprint y_arena_valve_controller:LED0805 -> y_arena_odor_controller:LED0805
- L10, L2, L3, L4, L5, L6, L7, L8, L9: footprint valve_spike_hold:LED0805 -> odor_spike_hold:LED0805
- MH1, MH2, MH3: footprint y_arena_valve_controller:MOUNTING_HOLE_4-40 -> y_arena_odor_controller:MOUNTING_HOLE_4-40
- P1: footprint y_arena_valve_controller:DCJACK_3PAD_SMD_RA -> y_arena_odor_controller:DCJACK_3PAD_SMD_RA
- R1: footprint y_arena_valve_controller:SM0402 -> y_arena_odor_controller:SM0402
- S1, S2, S3, S4, S5, S6, S7, S8, S9: footprint valve_spike_hold:LEECO_LHDB -> odor_spike_hold:LEECO_LHDB
- SW1: footprint y_arena_valve_controller:SPDT_SLIDE_500A_SM -> y_arena_odor_controller:SPDT_SLIDE_500A_SM
- TEENSY1: footprint y_arena_valve_controller:TEENSY_4.0 -> y_arena_odor_controller:TEENSY_4.0
- U1, U2, U3, U4, U5, U6, U7, U8, U9: footprint valve_spike_hold:SOIC_8 -> odor_spike_hold:SOIC_8
Connections:
- net /ARM_0_VALVE_0 renamed /ARM_0_ODOR_0
- net /ARM_0_VALVE_1 renamed /ARM_0_ODOR_1
- net /ARM_0_VALVE_2 renamed /ARM_0_ODOR_2
- net /ARM_1_VALVE_0 renamed /ARM_1_ODOR_0
- net /ARM_1_VALVE_1 renamed /ARM_1_ODOR_1
- net /ARM_1_VALVE_2 renamed /ARM_1_ODOR_2
- net /ARM_2_VALVE_0 renamed /ARM_2_ODOR_0
- net /ARM_2_VALVE_1 renamed /ARM_2_ODOR_1
- net /ARM_2_VALVE_2 renamed /ARM_2_ODOR_2
- net /valve_0/SH renamed /odor_0/SH
- net /valve_1/SH renamed /odor_1/SH
- net /valve_2/SH renamed /odor_2/SH
- net /valve_3/SH renamed /odor_3/SH
- net /valve_4/SH renamed /odor_4/SH
- net /valve_5/SH renamed /odor_5/SH
- net /valve_6/SH renamed /odor_6/SH
- net /valve_7/SH renamed /odor_7/SH
- net /valve_8/SH renamed /odor_8/SH
Other:
- rule pad_to_mask_clearance: 0.05 -> 0
- board text added: "ODOR"
- board text added: "ODOR 0"
- board text added: "ODOR 1"
- board text added: "ODOR 2"
- board text added: "y_arena_odor_controller Janelia Research Campus 10/2020 ver 1.3"
- board text removed: "VALVE"
- board text removed: "VALVE 0"
- board text removed: "VALVE 1"
- board text removed: "VALVE 2"
- board text removed: "y_arena_valve_controller Janelia Research Campus 07/31/2020 ver 1.2"
